Commit message: Revert axis for the tilt
Signed-off-by: Yehor Zvihunov <yehor.zvihunov@globallogic.com>

File: host-side/src/camera_description/urdf/camera-tilt.urdf.xacro (robot description, xacro)
@@ -74,5 +74,5 @@
       <child  link="${prefix}tilt_link"/>
       <origin xyz="0 0 0" rpy="0 0 0"/>
-      <axis xyz="0 0 1"/>
+      <axis xyz="0 0 -1"/>
       <limit lower="-3.1416" upper="3.1416" effort="5" velocity="3"/>
       <dynamics damping="0.1" friction="0.0"/>
@@ -104,9 +104,7 @@
       </inertial>
     </link>
-    <!-- камера жёстко прикручена к tilt -->
     <joint name="${prefix}camera_joint" type="revolute">
       <parent link="${prefix}tilt_link"/>
       <child  link="${prefix}camera_link"/>
-      <!-- cam_x/y/z подгони так, чтобы меш камеры встал на своё место -->
       <origin xyz="0 0 ${pivot_cam_z}" rpy="0 0 0"/>
       <axis xyz="1 0 0"/>
